Commit message: chore: apply git conventions and push workspace changes

File: urdf/base.urdf.xacro (robot description, xacro)
@@ -1,4 +1,4 @@
 <?xml version="1.0"?>
-<robot name="tetra" xmlns:xacro="http://www.ros.org/wiki/xacro">
+<robot name="robot" xmlns:xacro="http://www.ros.org/wiki/xacro">
   <!-- Define a number of dimensions using properties -->
   <xacro:property name="base_length" value="0.6127" />
@@ -23,5 +23,5 @@
     <origin xyz=" 0 ${-1.0*wheel_offset_y} 0 " rpy="0 0 0" />
 	<geometry>
-	  <mesh filename="package://tetra_gazebo_sim/meshes/wheel_drive_left.stl" scale="0.001 0.001 0.001" />
+	  <mesh filename="package://robot_gazebo_sim/meshes/wheel_drive_left.stl" scale="0.001 0.001 0.001" />
 	</geometry>
 	<material name="darkgrey"/>
@@ -50,5 +50,5 @@
     <origin xyz=" 0 ${wheel_offset_y} 0 " rpy="0 0 0" />
 	<geometry>
-	  <mesh filename="package://tetra_gazebo_sim/meshes/wheel_drive_right.stl" scale="0.001 0.001 0.001" />
+	  <mesh filename="package://robot_gazebo_sim/meshes/wheel_drive_right.stl" scale="0.001 0.001 0.001" />
 	</geometry>
 	<material name="darkgrey"/>
@@ -72,5 +72,5 @@
       <geometry>
         <mesh
-          filename="package://tetra_gazebo_sim/meshes/platform_body.stl" scale="0.001 0.001 0.001" />
+          filename="package://robot_gazebo_sim/meshes/platform_body.stl" scale="0.001 0.001 0.001" />
       </geometry>
       <material name="black"/>
@@ -107,5 +107,5 @@
                 <origin xyz="0 0 0" rpy="0 0 0"/>
                 <geometry>
-                    <mesh filename="package://tetra_gazebo_sim/meshes/caster_yoke.stl" scale="0.001 0.001 0.001" />
+                    <mesh filename="package://robot_gazebo_sim/meshes/caster_yoke.stl" scale="0.001 0.001 0.001" />
                 </geometry>
                 <material name="darkgrey" />
@@ -134,5 +134,5 @@
                 <origin xyz="0 0 0" rpy="0 0 0"/>
                 <geometry>
-                    <mesh filename="package://tetra_gazebo_sim/meshes/caster_wheel.stl" scale="0.001 0.001 0.001" />
+                    <mesh filename="package://robot_gazebo_sim/meshes/caster_wheel.stl" scale="0.001 0.001 0.001" />
                 </geometry>
                 <material name="darkgrey" />

File: urdf/tetra_base.xacro (robot description, xacro)
@@ -1,4 +1,4 @@
 <?xml version="1.0"?>
-<robot name="tetra" xmlns:xacro="http://www.ros.org/wiki/xacro">
+<robot name="robot" xmlns:xacro="http://www.ros.org/wiki/xacro">
   <!-- Define a number of dimensions using properties -->
   <xacro:property name="base_length" value="0.473" />
@@ -14,6 +14,6 @@
   </xacro:macro>
    <!-- Include all component files -->
-   <xacro:include filename="$(find tetra_gazebo_sim)/urdf/materials.urdf.xacro" />
-   <xacro:include filename="$(find tetra_gazebo_sim)/urdf/base.urdf.xacro" />
+   <xacro:include filename="$(find robot_gazebo_sim)/urdf/materials.urdf.xacro" />
+   <xacro:include filename="$(find robot_gazebo_sim)/urdf/base.urdf.xacro" />
    <!-- Add the base and wheels -->
    <base name="base" color="black"/>

File: urdf/tetra_gazebo.xacro (robot description, xacro)
@@ -1,6 +1,6 @@
 <?xml version="1.0"?>
-<robot name="tetra_gazebo" xmlns:xacro="http://www.ros.org/wiki/xacro">
-  <!-- Include the base tetra robot -->
-  <xacro:include filename="$(find tetra_gazebo_sim)/urdf/tetra_base.xacro" />
+<robot name="robot_gazebo" xmlns:xacro="http://www.ros.org/wiki/xacro">
+  <!-- Include the base robot robot -->
+  <xacro:include filename="$(find robot_gazebo_sim)/urdf/robot_base.xacro" />
   <!-- Gazebo colors -->
   <gazebo reference="base_link">
